File: 4channelPowerSupply/4channelPowerSupply.kicad_pcb (KiCad board)
At the start: 2 copper layers, 50 parts, among them J1 Input Voltage, J2 Output, Q1 DMP3013SFV, U1 LT8602EUJ#PBF

Commit message: Finished first project, yay
Parts:
- added REF**: OSHW-Logo2_14.6x12mm_SilkScreen, Symbol:OSHW-Logo2_14.6x12mm_SilkScreen, F.Cu at (162.8, 73.9)
- moved H4 83.1 mm to (203.2, 96.5)
- moved H1 81.6 mm to (157.5, 96.5)
- moved C1 73.9 mm to (176.3, 87.6), turned to 90 degrees
- moved C17 68.7 mm to (200.4, 79.9), turned to 270 degrees
- moved R9 67.2 mm to (175.9, 79.9), turned to 90 degrees
- moved C10 66.9 mm to (192.9, 83.1), turned to 270 degrees
- moved L3 66.6 mm to (194.6, 79.2), turned to 270 degrees
- moved C2 63.4 mm to (183.4, 87.6), turned to 90 degrees
- moved Q1 62.8 mm to (167.9, 89.5), turned to 180 degrees
- moved R1 60.7 mm to (170.2, 86.4)
- moved C11 60.5 mm to (199.0, 79.9), turned to 270 degrees
- moved C6 58.1 mm to (187.7, 69.5), turned to 270 degrees
- moved R14 57.9 mm to (165.7, 64.3), turned to 180 degrees
- moved J1 56.4 mm to (157.5, 84.5), turned to 270 degrees
- moved L4 55.5 mm to (179.6, 79.1), turned to 270 degrees
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- renumbered He to H1
Connections:
- J1 pad 1: VCC -> GND
- J1 pad 2: GND -> VCC
- J2 pad 1: +5V -> +1V8
- J2 pad 2: +3V3 -> +5V
- J2 pad 3: +1V8 -> +3V3
- U1 pad 1: (no net) -> Net-(U1-Pad1)
- U1 pad 12: (no net) -> Net-(U1-Pad12)
- U1 pad 31: (no net) -> Net-(U1-Pad31)
- U1 pad 32: (no net) -> Net-(U1-Pad32)
- U1 pad 40: (no net) -> Net-(U1-Pad40)
Routing:
- net +3V3: track 0.00 -> 94.1 mm, vias 0 -> 5
- net +1V8: track 0.00 -> 92.3 mm, vias 0 -> 1
- net +5V: track 0.00 -> 78.5 mm, vias 0 -> 1
- net +1V2: track 0.00 -> 53.0 mm
- net VCCQ: track 0.00 -> 45.8 mm, vias 0 -> 18
- net Net-(C13-Pad1): track 0.00 -> 35.4 mm, vias 0 -> 2
- net GND: track 0.00 -> 34.5 mm, vias 0 -> 61
- net Net-(C14-Pad1): track 0.00 -> 33.9 mm, vias 0 -> 2
- net Net-(C12-Pad1): track 0.00 -> 32.1 mm, vias 0 -> 2
- net Net-(C11-Pad1): track 0.00 -> 25.4 mm, vias 0 -> 2
- net Net-(R2-Pad1): track 0.00 -> 18.8 mm, vias 0 -> 3
- net VCC: track 0.00 -> 10.1 mm
- net Net-(C6-Pad1): track 0.00 -> 8.81 mm
- net Net-(C7-Pad1): track 0.00 -> 7.15 mm
- net Net-(L3-Pad1): track 0.00 -> 6.48 mm
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- added copper zone on B.Cu, net GND
- added copper zone on F.Cu, net GND
- added copper zone on In1.Cu, net GND
- added copper zone on In2.Cu, net VCCQ
Other:
- board outline added: 55.9 x 53.3 mm
- copper layers 2 -> 4
- board text added: "+1V2"
- board text added: "+1V8"
- board text added: "+3V3"
- board text added: "+5V"
- board text added: "- +"
- board text added: "1V2"
- board text added: "1V8"
- board text added: "3V3"
- board text added: "5V"
- board text added: "GND"
- board text added: "LT8602 - 4 CHANNEL POWER OUTPUT DESIGNED BY S.G. @ EMBDD - 2021"
