File: 4channelPowerSupply/4channelPowerSupply.sch (KiCad schematic (older format))
At the start: 50 parts, among them J1 Input Voltage, J2 Output, Q1 DMP3013SFV, U1 LT8602EUJ#PBF

Commit message: Finished first project, yay
Connections:
- net +1V8: now also J2.1 (Pin_1); no longer J2.3 (Pin_3)
- net +3V3: now also J2.3 (Pin_3); no longer J2.2 (Pin_2)
- net +5V: now also J2.2 (Pin_2); no longer J2.1 (Pin_1)
- net GND: now also J1.1 (Pin_1); no longer J1.2 (Pin_2)
- net VCC: now also J1.2 (Pin_2); no longer J1.1 (Pin_1)
Changed lines of the file:
@@
 Connection ~ 10050 5150
 $Comp
-L power:+5V #PWR0120
-U 1 1 60C835CB
+L power:+3.3V #PWR0121
+U 1 1 60C83D20
+P 1650 1450
+F 0 "#PWR0121" H 1650 1300 50  0001 C CNN
+F 1 "+3.3V" V 1650 1700 50  0000 C CNN
+F 2 "" H 1650 1450 50  0001 C CNN
+F 3 "" H 1650 1450 50  0001 C CNN
+	1    1650 1450
+	-1   0    0    1
+$EndComp
+$Comp
+L power:+1V8 #PWR0122
+U 1 1 60C845FD
 P 1450 1450
-F 0 "#PWR0120" H 1450 1300 50  0001 C CNN
-F 1 "+5V" V 1450 1700 50  0000 C CNN
+F 0 "#PWR0122" H 1450 1300 50  0001 C CNN
+F 1 "+1V8" V 1450 1700 50  0000 C CNN
 F 2 "" H 1450 1450 50  0001 C CNN
 F 3 "" H 1450 1450 50  0001 C CNN
 	1    1450 1450
-	-1   0    0    1
-$EndComp
-$Comp
-L power:+3.3V #PWR0121
-U 1 1 60C83D20
-P 1550 1450
-F 0 "#PWR0121" H 1550 1300 50  0001 C CNN
-F 1 "+3.3V" V 1550 1700 50  0000 C CNN
-F 2 "" H 1550 1450 50  0001 C CNN
-F 3 "" H 1550 1450 50  0001 C CNN
-	1    1550 1450
-	-1   0    0    1
-$EndComp
-$Comp
-L power:+1V8 #PWR0122
-U 1 1 60C845FD
-P 1650 1450
-F 0 "#PWR0122" H 1650 1300 50  0001 C CNN
-F 1 "+1V8" V 1650 1700 50  0000 C CNN
-F 2 "" H 1650 1450 50  0001 C CNN
-F 3 "" H 1650 1450 50  0001 C CNN
-	1    1650 1450
 	-1   0    0    1
 $EndComp
@@
 L power:VCC #PWR0125
 U 1 1 60C86411
+P 1050 1450
+F 0 "#PWR0125" H 1050 1300 50  0001 C CNN
+F 1 "VCC" V 1050 1650 50  0000 C CNN
+F 2 "" H 1050 1450 50  0001 C CNN
+F 3 "" H 1050 1450 50  0001 C CNN
+	1    1050 1450
+	-1   0    0    1
+$EndComp
+$Comp
+L power:GND #PWR0126
+U 1 1 60C87399
 P 950 1450
-F 0 "#PWR0125" H 950 1300 50  0001 C CNN
-F 1 "VCC" V 950 1650 50  0000 C CNN
+F 0 "#PWR0126" H 950 1200 50  0001 C CNN
+F 1 "GND" V 950 1250 50  0000 C CNN
 F 2 "" H 950 1450 50  0001 C CNN
 F 3 "" H 950 1450 50  0001 C CNN
 	1    950  1450
-	-1   0    0    1
-$EndComp
-$Comp
-L power:GND #PWR0126
-U 1 1 60C87399
-P 1050 1450
-F 0 "#PWR0126" H 1050 1200 50  0001 C CNN
-F 1 "GND" V 1050 1250 50  0000 C CNN
-F 2 "" H 1050 1450 50  0001 C CNN
-F 3 "" H 1050 1450 50  0001 C CNN
-	1    1050 1450
 	1    0    0    -1
 $EndComp
@@
 Text Notes 2900 4500 0    118  ~ 24
 POWER INDICATION\n
+$Comp
+L power:+5V #PWR0120
+U 1 1 60C835CB
+P 1550 1450
+F 0 "#PWR0120" H 1550 1300 50  0001 C CNN
+F 1 "+5V" V 1550 1700 50  0000 C CNN
+F 2 "" H 1550 1450 50  0001 C CNN
+F 3 "" H 1550 1450 50  0001 C CNN
+	1    1550 1450
+	-1   0    0    1
+$EndComp
 $EndSCHEMATC
