File: servoController/servoController.sch (KiCad schematic (older format))
At the start: 43 parts

Commit message: Servocontroller
Parts:
- added D2: LED, LED_SMD:LED_0402_1005Metric, symbol Device:LED
- added H1, H2, H3, H4: MountingHole, MountingHole:MountingHole_2.1mm, symbol Mechanical:MountingHole
- added R10: 10K, Resistor_SMD:R_0402_1005Metric, symbol Device:R
- J3: renamed from J?; symbol Connector_Generic:Conn_02x04_Counter_Clockwise -> Connector_Generic:Conn_02x04_Odd_Even
- gave numbers to parts that had none: 42
Connections:
- net +3V3: now also J3.2 (Pin_2), R10.1; no longer J3.8 (Pin_8)
- net CAN_H: now also J1.2 (Pin_2); no longer J1.3 (Pin_3)
- net CAN_L: now also J1.3 (Pin_3); no longer J1.2 (Pin_2)
- net ENC_1: now also J3.3 (Pin_3); no longer J3.2 (Pin_2)
- net ENC_2: now also J3.5 (Pin_5); no longer J3.3 (Pin_3)
- net GND: now also J3.7 (Pin_7), J3.8 (Pin_8); no longer J3.4 (Pin_4), J3.5 (Pin_5)
- net LMT_SW1: now also J3.4 (Pin_4); no longer J3.7 (Pin_7)
- net MTR_ENABLE: now also U3.4 (ENABLE)
- net MTR_MODE1: now also U3.16 (MODE1)
- net MTR_MODE2: now also U3.5 (MODE2)
- net MTR_PHASE: now also U3.1 (PHASE)
- net MTR_SLEEP: now also U3.3 (~SLEEP)
- net OSC1: now also U4.5 (PD0)
- net OSC2: now also U4.6 (PD1)
- net RTCOSC1: now also U4.3 (PC14)
- net RTCOSC2: now also U4.4 (PC15)
- net SCL: now also J1.4 (Pin_4), R8.2; no longer J1.5 (Pin_5), R7.2
- net SDA: now also J1.5 (Pin_5), R7.2; no longer J1.4 (Pin_4), R8.2
- net at U4.2 (PC13): now also D2.1 (K)
- new net: D2.2 (A), R10.2
Other:
- note added: "CAN Bus driver"
- note added: "Crystals"
- note added: "Encoder and limit switch \nconnector"
- note added: "I2C, Reset, Decoupling\n"
- note added: "MCU connectors"
- note added: "Main Connector"
- note added: "Motor driver\n"
- note added: "Mouting Holes\n"
- note added: "Power"
- note added: "STM32F103C8"
- moved on the sheet: C1, C10, C11, C12, C13, C14, C15, C16, C17, C18, C19, C2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
